Commit message: add visualization mode and single arm mode

File: husky_panda_description/urdf/husky.urdf.xacro (robot description, xacro)
@@ -32,5 +32,4 @@
   <xacro:property name="husky_rear_bumper_extend" value="$(optenv HUSKY_REAR_BUMPER_EXTEND 0)" />
   <xacro:arg name="robot_namespace" default="/" />
-  <xacro:arg name="urdf_extras" default="empty.urdf" />
   <!-- Included URDF/XACRO Files -->
   <xacro:include filename="$(find husky_description)/urdf/decorations.urdf.xacro" />
@@ -182,5 +181,4 @@
   </gazebo>
   <!-- Optional custom includes. -->
-  <xacro:include filename="$(arg urdf_extras)" />
   <xacro:include filename="$(find roas_bringup)/urdf/roas.urdf.xacro"/>
 </robot>

File: husky_panda_description/urdf/husky_panda.urdf.xacro (robot description, xacro)
@@ -3,15 +3,25 @@
     <xacro:arg name="robot_namespace" default="/" />
     <xacro:arg name="single_arm" default="true"/>
-    <xacro:arg name="arm_id" default="panda" />
-    <!-- Should a franka_gripper be mounted at the flange?" -->
-    <xacro:arg name="hand" default="true" />
     <!-- Is the robot being simulated in gazebo?" -->
-    <xacro:arg name="gazebo" default="true" />
+    <xacro:arg name="gazebo" default="false" />
     <xacro:arg name="connected_to" default=" "/>
+    <xacro:arg name="x"     default="0"/>
+    <xacro:arg name="y"     default="0"/>
+    <xacro:arg name="z"     default="0"/>
+    <xacro:arg name="roll"  default="0"/>
+    <xacro:arg name="pitch" default="0"/>
+    <xacro:arg name="yaw"   default="0"/>
     <xacro:include filename="$(find husky_panda_description)/urdf/husky.urdf.xacro"/>
     <xacro:include filename="$(find husky_panda_description)/urdf/panda_arm.urdf.xacro"/>
     <xacro:if value="$(arg single_arm)">
+        <xacro:arg name="arm_id" default="panda" />
+        <xacro:panda arm_id="$(arg arm_id)" gazebo="$(arg gazebo)" connected_to="$(arg connected_to)" x="$(arg x)" y="$(arg y)" z="$(arg z)" roll="$(arg roll)" pitch="$(arg pitch)" yaw="$(arg yaw)">
+        </xacro:panda>
     </xacro:if>
     <xacro:unless value="$(arg single_arm)">
+        <xacro:arg name="arm_id_1" default="panda_1" />
+        <xacro:arg name="arm_id_2" default="panda_2" />
+        <xacro:panda arm_id="$(arg arm_id_1)" gazebo="$(arg gazebo)" connected_to="$(arg connected_to)" x="$(arg x)" y="$(arg y)" z="$(arg z)" roll="$(arg roll)" pitch="$(arg pitch)" yaw="$(arg yaw)"/>
+        <xacro:panda arm_id="$(arg arm_id_2)" gazebo="$(arg gazebo)" connected_to="$(arg connected_to)" x="$(arg x)" y="-$(arg y)" z="$(arg z)" roll="$(arg roll)" pitch="$(arg pitch)" yaw="$(arg yaw)"/>
     </xacro:unless>
 </robot>

File: husky_panda_description/urdf/panda_arm.urdf.xacro (robot description, xacro)
@@ -1,67 +1,61 @@
 <?xml version='1.0' encoding='utf-8'?>
 <robot xmlns:xacro="http://www.ros.org/wiki/xacro" name="panda">
-  <!-- Name of this panda -->
-  <xacro:arg name="arm_id" default="panda" />
+  <xacro:macro name="panda" params="arm_id:='panda' gazebo:='' connected_to:='' x=0 y=0 z=0 roll=0 pitch=0 yaw=0">
   <!-- Should a franka_gripper be mounted at the flange?" -->
-  <xacro:arg name="hand" default="false" />
-  <!-- Is the robot being simulated in gazebo?" -->
-  <xacro:arg name="gazebo" default="false" />
-  <xacro:arg name="connected_to" default=" "/>
-  <xacro:unless value="$(arg gazebo)">
+  <xacro:arg name="hand" default="true" />
+  <xacro:unless value="${gazebo}">
     <!-- Create a URDF for a real hardware -->
     <xacro:include filename="$(find franka_description)/robots/panda_arm.xacro" />
-    <xacro:panda_arm arm_id="$(arg arm_id)" safety_distance="0.03"/>
+    <xacro:panda_arm arm_id="${arm_id}" safety_distance="0.03"/>
     <xacro:if value="$(arg hand)">
       <xacro:include filename="$(find franka_description)/robots/hand.xacro"/>
-      <xacro:hand arm_id="$(arg arm_id)" rpy="0 0 ${-pi/4}" connected_to="$(arg arm_id)_link8" safety_distance="0.03"/>
+      <xacro:hand arm_id="${arm_id}" rpy="0 0 ${-pi/4}" connected_to="${arm_id}_link8" safety_distance="0.03"/>
     </xacro:if>
   </xacro:unless>
-  <xacro:if value="$(arg gazebo)">
-    <xacro:arg name="xyz" default="0 0 0" />
-    <xacro:arg name="rpy" default="0 0 0" />
+  <xacro:if value="${gazebo}">
     <!-- Create a simulatable URDF -->
     <xacro:include filename="$(find franka_description)/robots/utils.xacro" />
     <xacro:include filename="$(find franka_description)/robots/panda_gazebo.xacro" />
-    <xacro:panda_arm arm_id="$(arg arm_id)" connected_to="$(arg connected_to)"/>
+    <xacro:panda_arm arm_id="${arm_id}" connected_to="${connected_to}"/>
     <xacro:if value="$(arg hand)">
-      <xacro:hand arm_id="$(arg arm_id)" rpy="0 0 ${-pi/4}" connected_to="$(arg arm_id)_link8" />
-      <xacro:gazebo-joint joint="$(arg arm_id)_finger_joint1" transmission="hardware_interface/EffortJointInterface" />
-      <xacro:gazebo-joint joint="$(arg arm_id)_finger_joint2" transmission="hardware_interface/EffortJointInterface" />
+      <xacro:hand arm_id="${arm_id}" rpy="0 0 ${-pi/4}" connected_to="${arm_id}_link8" />
+      <xacro:gazebo-joint joint="${arm_id}_finger_joint1" transmission="hardware_interface/EffortJointInterface" />
+      <xacro:gazebo-joint joint="${arm_id}_finger_joint2" transmission="hardware_interface/EffortJointInterface" />
     </xacro:if>
     <!-- Gazebo requires a joint to a link called "world" for statically mounted robots -->
-    <link name="world" />
-    <joint name="world_joint" type="fixed">
-      <origin xyz="$(arg xyz)" rpy="$(arg rpy)" />
-      <parent link="world" />
-      <child  link="$(arg arm_id)_link0" />
+    <joint name="${connected_to}_to_${arm_id}_joint" type="fixed">
+      <origin xyz="${x} ${y} ${z}" rpy="${roll} ${pitch} ${yaw}" />
+      <parent link="${connected_to}" />
+      <child  link="${arm_id}_link0" />
     </joint>
-    <xacro:gazebo-joint joint="$(arg arm_id)_joint1" transmission="hardware_interface/PositionJointInterface" />
-    <xacro:gazebo-joint joint="$(arg arm_id)_joint2" transmission="hardware_interface/PositionJointInterface" />
-    <xacro:gazebo-joint joint="$(arg arm_id)_joint3" transmission="hardware_interface/PositionJointInterface" />
-    <xacro:gazebo-joint joint="$(arg arm_id)_joint4" transmission="hardware_interface/PositionJointInterface" />
-    <xacro:gazebo-joint joint="$(arg arm_id)_joint5" transmission="hardware_interface/PositionJointInterface" />
-    <xacro:gazebo-joint joint="$(arg arm_id)_joint6" transmission="hardware_interface/PositionJointInterface" />
-    <xacro:gazebo-joint joint="$(arg arm_id)_joint7" transmission="hardware_interface/PositionJointInterface" />
-    <xacro:gazebo-joint joint="$(arg arm_id)_joint1" transmission="hardware_interface/VelocityJointInterface" />
-    <xacro:gazebo-joint joint="$(arg arm_id)_joint2" transmission="hardware_interface/VelocityJointInterface" />
-    <xacro:gazebo-joint joint="$(arg arm_id)_joint3" transmission="hardware_interface/VelocityJointInterface" />
-    <xacro:gazebo-joint joint="$(arg arm_id)_joint4" transmission="hardware_interface/VelocityJointInterface" />
-    <xacro:gazebo-joint joint="$(arg arm_id)_joint5" transmission="hardware_interface/VelocityJointInterface" />
-    <xacro:gazebo-joint joint="$(arg arm_id)_joint6" transmission="hardware_interface/VelocityJointInterface" />
-    <xacro:gazebo-joint joint="$(arg arm_id)_joint7" transmission="hardware_interface/VelocityJointInterface" />
-    <xacro:gazebo-joint joint="$(arg arm_id)_joint1" transmission="hardware_interface/EffortJointInterface" />
-    <xacro:gazebo-joint joint="$(arg arm_id)_joint2" transmission="hardware_interface/EffortJointInterface" />
-    <xacro:gazebo-joint joint="$(arg arm_id)_joint3" transmission="hardware_interface/EffortJointInterface" />
-    <xacro:gazebo-joint joint="$(arg arm_id)_joint4" transmission="hardware_interface/EffortJointInterface" />
-    <xacro:gazebo-joint joint="$(arg arm_id)_joint5" transmission="hardware_interface/EffortJointInterface" />
-    <xacro:gazebo-joint joint="$(arg arm_id)_joint6" transmission="hardware_interface/EffortJointInterface" />
-    <xacro:gazebo-joint joint="$(arg arm_id)_joint7" transmission="hardware_interface/EffortJointInterface" />
-    <xacro:transmission-franka-state arm_id="$(arg arm_id)" />
-    <xacro:transmission-franka-model arm_id="$(arg arm_id)"
-       root="$(arg arm_id)_joint1"
-       tip="$(arg arm_id)_joint8"
+    <xacro:gazebo-joint joint="${arm_id}_joint1" transmission="hardware_interface/PositionJointInterface" />
+    <xacro:gazebo-joint joint="${arm_id}_joint2" transmission="hardware_interface/PositionJointInterface" />
+    <xacro:gazebo-joint joint="${arm_id}_joint3" transmission="hardware_interface/PositionJointInterface" />
+    <xacro:gazebo-joint joint="${arm_id}_joint4" transmission="hardware_interface/PositionJointInterface" />
+    <xacro:gazebo-joint joint="${arm_id}_joint5" transmission="hardware_interface/PositionJointInterface" />
+    <xacro:gazebo-joint joint="${arm_id}_joint6" transmission="hardware_interface/PositionJointInterface" />
+    <xacro:gazebo-joint joint="${arm_id}_joint7" transmission="hardware_interface/PositionJointInterface" />
+    <xacro:gazebo-joint joint="${arm_id}_joint1" transmission="hardware_interface/VelocityJointInterface" />
+    <xacro:gazebo-joint joint="${arm_id}_joint2" transmission="hardware_interface/VelocityJointInterface" />
+    <xacro:gazebo-joint joint="${arm_id}_joint3" transmission="hardware_interface/VelocityJointInterface" />
+    <xacro:gazebo-joint joint="${arm_id}_joint4" transmission="hardware_interface/VelocityJointInterface" />
+    <xacro:gazebo-joint joint="${arm_id}_joint5" transmission="hardware_interface/VelocityJointInterface" />
+    <xacro:gazebo-joint joint="${arm_id}_joint6" transmission="hardware_interface/VelocityJointInterface" />
+    <xacro:gazebo-joint joint="${arm_id}_joint7" transmission="hardware_interface/VelocityJointInterface" />
+    <xacro:gazebo-joint joint="${arm_id}_joint1" transmission="hardware_interface/EffortJointInterface" />
+    <xacro:gazebo-joint joint="${arm_id}_joint2" transmission="hardware_interface/EffortJointInterface" />
+    <xacro:gazebo-joint joint="${arm_id}_joint3" transmission="hardware_interface/EffortJointInterface" />
+    <xacro:gazebo-joint joint="${arm_id}_joint4" transmission="hardware_interface/EffortJointInterface" />
+    <xacro:gazebo-joint joint="${arm_id}_joint5" transmission="hardware_interface/EffortJointInterface" />
+    <xacro:gazebo-joint joint="${arm_id}_joint6" transmission="hardware_interface/EffortJointInterface" />
+    <xacro:gazebo-joint joint="${arm_id}_joint7" transmission="hardware_interface/EffortJointInterface" />
+    <xacro:transmission-franka-state arm_id="${arm_id}" />
+    <xacro:transmission-franka-model arm_id="${arm_id}"
+       root="${arm_id}_joint1"
+       tip="${arm_id}_joint8"
      />
     <gazebo>
       <plugin name="gazebo_ros_control" filename="libgazebo_ros_control.so">
+        <robotNamespace>${arm_id}</robotNamespace>
         <controlPeriod>0.001</controlPeriod>
         <robotSimType>franka_gazebo/FrankaHWSim</robotSimType>
@@ -70,3 +64,4 @@
     </gazebo>
   </xacro:if>
+  </xacro:macro>
 </robot>
