Commit message: set the default option of gazebo to false

File: husky_panda_description/urdf/husky_panda.urdf.xacro (robot description, xacro)
@@ -16,6 +16,5 @@
     <xacro:if value="$(arg single_arm)">
         <xacro:arg name="arm_id" default="panda" />
-        <xacro:panda arm_id="$(arg arm_id)" gazebo="$(arg gazebo)" connected_to="$(arg connected_to)" x="$(arg x)" y="$(arg y)" z="$(arg z)" roll="$(arg roll)" pitch="$(arg pitch)" yaw="$(arg yaw)">
-        </xacro:panda>
+        <xacro:panda arm_id="$(arg arm_id)" gazebo="$(arg gazebo)" connected_to="$(arg connected_to)" x="$(arg x)" y="$(arg y)" z="$(arg z)" roll="$(arg roll)" pitch="$(arg pitch)" yaw="$(arg yaw)"/>
     </xacro:if>
     <xacro:unless value="$(arg single_arm)">

File: husky_panda_description/urdf/panda_arm.urdf.xacro (robot description, xacro)
@@ -7,5 +7,5 @@
     <!-- Create a URDF for a real hardware -->
     <xacro:include filename="$(find franka_description)/robots/panda_arm.xacro" />
-    <xacro:panda_arm arm_id="${arm_id}" safety_distance="0.03"/>
+    <xacro:panda_arm arm_id="${arm_id}" safety_distance="0.03" connected_to="${connected_to}"/>
     <xacro:if value="$(arg hand)">
       <xacro:include filename="$(find franka_description)/robots/hand.xacro"/>
@@ -17,5 +17,5 @@
     <xacro:include filename="$(find franka_description)/robots/utils.xacro" />
     <xacro:include filename="$(find franka_description)/robots/panda_gazebo.xacro" />
-    <xacro:panda_arm arm_id="${arm_id}" connected_to="${connected_to}"/>
+    <xacro:panda_arm arm_id="${arm_id}" connected_to="${connected_to}" xyz="${x} ${y} ${z}" rpy="${roll} ${pitch} ${yaw}"/>
     <xacro:if value="$(arg hand)">
       <xacro:hand arm_id="${arm_id}" rpy="0 0 ${-pi/4}" connected_to="${arm_id}_link8" />
@@ -23,10 +23,4 @@
       <xacro:gazebo-joint joint="${arm_id}_finger_joint2" transmission="hardware_interface/EffortJointInterface" />
     </xacro:if>
-    <!-- Gazebo requires a joint to a link called "world" for statically mounted robots -->
-    <joint name="${connected_to}_to_${arm_id}_joint" type="fixed">
-      <origin xyz="${x} ${y} ${z}" rpy="${roll} ${pitch} ${yaw}" />
-      <parent link="${connected_to}" />
-      <child  link="${arm_id}_link0" />
-    </joint>
     <xacro:gazebo-joint joint="${arm_id}_joint1" transmission="hardware_interface/PositionJointInterface" />
     <xacro:gazebo-joint joint="${arm_id}_joint2" transmission="hardware_interface/PositionJointInterface" />
