Commit message: update a first version

File: husky_panda_manipulation/data/panda.urdf.xacro (robot description, xacro)
@@ -21,5 +21,5 @@
         <xacro:panda_robot parent_link="world"/>
     </xacro:if>
-    <!-- Add a omnidirectional base to the robot -->
+    <!-- Add a mobile base to the robot -->
     <xacro:unless value="${fixed_base}">
         <link name="world"/>

File: husky_panda_manipulation/data/planar_base.urdf.xacro (robot description, xacro)
@@ -14,5 +14,5 @@
     </xacro:macro>
     <xacro:macro name="planar_base" params="connect_to">
-        <link name="omni_base_root_link"/>
+        <link name="husky_base_root_link"/>
         <link name="x_slider">
             <inertial>
@@ -37,5 +37,5 @@
         </link>
         <joint name="x_base_joint" type="prismatic">
-            <parent link="omni_base_root_link"/>
+            <parent link="husky_base_root_link"/>
             <child link="x_slider"/>
             <origin rpy="0 0 0" xyz="0.0 0.0 0.0"/>
@@ -63,5 +63,5 @@
         </joint>
         <xacro:add_transmission joint_name="pivot_joint"/>
-        <joint name="omni_base_flange" type="fixed">
+        <joint name="husky_base_flange" type="fixed">
             <parent link="pivot"/>
             <child link="${connect_to}"/>
