Commit message: increase the height of base_link

File: husky_panda_manipulation/data/planar_base.urdf.xacro (robot description, xacro)
@@ -66,4 +66,5 @@
             <parent link="pivot"/>
             <child link="${connect_to}"/>
+            <origin xyz="0 0 0.13228" rpy="0 0 0" />
         </joint>
     </xacro:macro>
