Commit message: update a package

File: husky_panda_manipulation/data/husky.urdf.xacro (robot description, xacro)
@@ -55,4 +55,5 @@
   <xacro:arg name="urdf_extras" default="$(optenv HUSKY_URDF_EXTRAS empty.urdf)" />
   <xacro:arg name="cpr_urdf_extras" default="$(optenv CPR_URDF_EXTRAS empty.urdf)" />
+  <xacro:property name="fixed_wheel" default="${False}" />
   <!-- Included URDF/XACRO Files -->
   <xacro:include filename="$(find husky_panda_manipulation)/data/decorations.urdf.xacro" />
@@ -127,14 +128,14 @@
   </gazebo>
   <!-- Husky wheel macros -->
-  <xacro:husky_wheel wheel_prefix="front_left">
+  <xacro:husky_wheel wheel_prefix="front_left" fixed_wheel="${fixed_wheel}">
     <origin xyz="${wheelbase/2} ${track/2} ${wheel_vertical_offset}" rpy="0 0 0" />
   </xacro:husky_wheel>
-  <xacro:husky_wheel wheel_prefix="front_right">
+  <xacro:husky_wheel wheel_prefix="front_right" fixed_wheel="${fixed_wheel}">
     <origin xyz="${wheelbase/2} ${-track/2} ${wheel_vertical_offset}" rpy="0 0 0" />
   </xacro:husky_wheel>
-  <xacro:husky_wheel wheel_prefix="rear_left">
+  <xacro:husky_wheel wheel_prefix="rear_left" fixed_wheel="${fixed_wheel}">
     <origin xyz="${-wheelbase/2} ${track/2} ${wheel_vertical_offset}" rpy="0 0 0" />
   </xacro:husky_wheel>
-  <xacro:husky_wheel wheel_prefix="rear_right">
+  <xacro:husky_wheel wheel_prefix="rear_right" fixed_wheel="${fixed_wheel}">
     <origin xyz="${-wheelbase/2} ${-track/2} ${wheel_vertical_offset}" rpy="0 0 0" />
   </xacro:husky_wheel>

File: husky_panda_manipulation/data/wheel.urdf.xacro (robot description, xacro)
@@ -22,5 +22,5 @@
 -->
 <robot xmlns:xacro="http://ros.org/wiki/xacro" name="husky_wheel">
-	<xacro:macro name="husky_wheel" params="wheel_prefix *joint_pose">
+	<xacro:macro name="husky_wheel" params="fixed_wheel wheel_prefix *joint_pose">
 		<link name="${wheel_prefix}_wheel_link">
 			<inertial>
@@ -49,5 +49,6 @@
 			<fdir1 value="1 0 0"/>
 		</gazebo>
-		<joint name="${wheel_prefix}_wheel" type="fixed">
+	      <xacro:unless value="${fixed_wheel}">
+			<joint name="${wheel_prefix}_wheel" type="fixed">
 			<parent link="base_link"/>
 			<child link="${wheel_prefix}_wheel_link"/>
@@ -55,19 +56,22 @@
 			<axis xyz="0 1 0" rpy="0 0 0" />
 		</joint>
-		<!-- <joint name="${wheel_prefix}_wheel" type="continuous">
-			<parent link="base_link"/>
-			<child link="${wheel_prefix}_wheel_link"/>
-			<xacro:insert_block name="joint_pose"/>
-			<axis xyz="0 1 0" rpy="0 0 0" />
-		</joint>
-		<transmission name="${wheel_prefix}_wheel_trans" type="SimpleTransmission">
-			<type>transmission_interface/SimpleTransmission</type>
-			<actuator name="${wheel_prefix}_wheel_motor">
-				<mechanicalReduction>1</mechanicalReduction>
-			</actuator>
-			<joint name="${wheel_prefix}_wheel">
-				<hardwareInterface>hardware_interface/VelocityJointInterface</hardwareInterface>
+	      </xacro:unless>
+		<xacro:if value="${fixed_wheel}">
+			<joint name="${wheel_prefix}_wheel" type="continuous">
+				<parent link="base_link"/>
+				<child link="${wheel_prefix}_wheel_link"/>
+				<xacro:insert_block name="joint_pose"/>
+				<axis xyz="0 1 0" rpy="0 0 0" />
 			</joint>
-		</transmission> -->
+			<transmission name="${wheel_prefix}_wheel_trans" type="SimpleTransmission">
+				<type>transmission_interface/SimpleTransmission</type>
+				<actuator name="${wheel_prefix}_wheel_motor">
+					<mechanicalReduction>1</mechanicalReduction>
+				</actuator>
+				<joint name="${wheel_prefix}_wheel">
+					<hardwareInterface>hardware_interface/VelocityJointInterface</hardwareInterface>
+				</joint>
+			</transmission>
+	      </xacro:if>
 	</xacro:macro>
 </robot>

Commit message: modify husky wheel models

File: husky_panda_manipulation/data/husky.urdf.xacro (robot description, xacro)
@@ -55,5 +55,4 @@
   <xacro:arg name="urdf_extras" default="$(optenv HUSKY_URDF_EXTRAS empty.urdf)" />
   <xacro:arg name="cpr_urdf_extras" default="$(optenv CPR_URDF_EXTRAS empty.urdf)" />
-  <xacro:property name="fixed_wheel" default="${False}" />
   <!-- Included URDF/XACRO Files -->
   <xacro:include filename="$(find husky_panda_manipulation)/data/decorations.urdf.xacro" />
@@ -128,14 +127,14 @@
   </gazebo>
   <!-- Husky wheel macros -->
-  <xacro:husky_wheel wheel_prefix="front_left" fixed_wheel="${fixed_wheel}">
+  <xacro:husky_wheel wheel_prefix="front_left">
     <origin xyz="${wheelbase/2} ${track/2} ${wheel_vertical_offset}" rpy="0 0 0" />
   </xacro:husky_wheel>
-  <xacro:husky_wheel wheel_prefix="front_right" fixed_wheel="${fixed_wheel}">
+  <xacro:husky_wheel wheel_prefix="front_right">
     <origin xyz="${wheelbase/2} ${-track/2} ${wheel_vertical_offset}" rpy="0 0 0" />
   </xacro:husky_wheel>
-  <xacro:husky_wheel wheel_prefix="rear_left" fixed_wheel="${fixed_wheel}">
+  <xacro:husky_wheel wheel_prefix="rear_left">
     <origin xyz="${-wheelbase/2} ${track/2} ${wheel_vertical_offset}" rpy="0 0 0" />
   </xacro:husky_wheel>
-  <xacro:husky_wheel wheel_prefix="rear_right" fixed_wheel="${fixed_wheel}">
+  <xacro:husky_wheel wheel_prefix="rear_right">
     <origin xyz="${-wheelbase/2} ${-track/2} ${wheel_vertical_offset}" rpy="0 0 0" />
   </xacro:husky_wheel>

File: husky_panda_manipulation/data/wheel.urdf.xacro (robot description, xacro)
@@ -22,5 +22,5 @@
 -->
 <robot xmlns:xacro="http://ros.org/wiki/xacro" name="husky_wheel">
-	<xacro:macro name="husky_wheel" params="fixed_wheel wheel_prefix *joint_pose">
+	<xacro:macro name="husky_wheel" params="wheel_prefix *joint_pose">
 		<link name="${wheel_prefix}_wheel_link">
 			<inertial>
@@ -49,6 +49,5 @@
 			<fdir1 value="1 0 0"/>
 		</gazebo>
-	      <xacro:unless value="${fixed_wheel}">
-			<joint name="${wheel_prefix}_wheel" type="fixed">
+		<joint name="${wheel_prefix}_wheel" type="fixed">
 			<parent link="base_link"/>
 			<child link="${wheel_prefix}_wheel_link"/>
@@ -56,22 +55,19 @@
 			<axis xyz="0 1 0" rpy="0 0 0" />
 		</joint>
-	      </xacro:unless>
-		<xacro:if value="${fixed_wheel}">
-			<joint name="${wheel_prefix}_wheel" type="continuous">
-				<parent link="base_link"/>
-				<child link="${wheel_prefix}_wheel_link"/>
-				<xacro:insert_block name="joint_pose"/>
-				<axis xyz="0 1 0" rpy="0 0 0" />
+		<!-- <joint name="${wheel_prefix}_wheel" type="continuous">
+			<parent link="base_link"/>
+			<child link="${wheel_prefix}_wheel_link"/>
+			<xacro:insert_block name="joint_pose"/>
+			<axis xyz="0 1 0" rpy="0 0 0" />
+		</joint>
+		<transmission name="${wheel_prefix}_wheel_trans" type="SimpleTransmission">
+			<type>transmission_interface/SimpleTransmission</type>
+			<actuator name="${wheel_prefix}_wheel_motor">
+				<mechanicalReduction>1</mechanicalReduction>
+			</actuator>
+			<joint name="${wheel_prefix}_wheel">
+				<hardwareInterface>hardware_interface/VelocityJointInterface</hardwareInterface>
 			</joint>
-			<transmission name="${wheel_prefix}_wheel_trans" type="SimpleTransmission">
-				<type>transmission_interface/SimpleTransmission</type>
-				<actuator name="${wheel_prefix}_wheel_motor">
-					<mechanicalReduction>1</mechanicalReduction>
-				</actuator>
-				<joint name="${wheel_prefix}_wheel">
-					<hardwareInterface>hardware_interface/VelocityJointInterface</hardwareInterface>
-				</joint>
-			</transmission>
-	      </xacro:if>
+		</transmission> -->
 	</xacro:macro>
 </robot>
