Commit message: update husky_panda_manipulation

File: husky_panda_manipulation/data/husky_panda_mobile.urdf.xacro (robot description, xacro)
@@ -9,9 +9,14 @@
     <!-- husky base -->
     <xacro:unless value="$(arg fixed_base)">
+        <link name="husky_base_root_link"/>
         <joint name="world_joint" type="fixed">
             <parent link="world"/>
             <child link="husky_base_root_link"/>
         </joint>
-        <xacro:planar_base connect_to="base_link"/>
+        <joint name="husky_base_flange" type="fixed">
+            <parent link="husky_base_root_link"/>
+            <child link="base_link"/>
+            <origin xyz="0 0 0.13228" rpy="0 0 0" />
+        </joint>
     </xacro:unless>
     <xacro:if value="$(arg fixed_base)">

File: husky_panda_manipulation/data/wheel.urdf.xacro (robot description, xacro)
@@ -49,11 +49,5 @@
 			<fdir1 value="1 0 0"/>
 		</gazebo>
-		<joint name="${wheel_prefix}_wheel" type="fixed">
-			<parent link="base_link"/>
-			<child link="${wheel_prefix}_wheel_link"/>
-			<xacro:insert_block name="joint_pose"/>
-			<axis xyz="0 1 0" rpy="0 0 0" />
-		</joint>
-		<!-- <joint name="${wheel_prefix}_wheel" type="continuous">
+		<joint name="${wheel_prefix}_wheel" type="continuous">
 			<parent link="base_link"/>
 			<child link="${wheel_prefix}_wheel_link"/>
@@ -69,5 +63,5 @@
 				<hardwareInterface>hardware_interface/VelocityJointInterface</hardwareInterface>
 			</joint>
-		</transmission> -->
+		</transmission>
 	</xacro:macro>
 </robot>

Commit message: modify models from holonomic to non-holonomic

File: husky_panda_manipulation/data/husky_panda_mobile.urdf.xacro (robot description, xacro)
@@ -3,20 +3,20 @@
     <xacro:arg name="fixed_base" default="false"/>
     <xacro:include filename="$(find mppi_panda)/resources/panda/panda.urdf.xacro"/>
-    <xacro:include filename="$(find husky_panda_manipulation)/data/planar_base.urdf.xacro"/>
+    <!-- <xacro:include filename="$(find husky_panda_manipulation)/data/planar_base.urdf.xacro"/> -->
     <xacro:include filename="$(find husky_panda_manipulation)/data/husky.urdf.xacro"/>
     <!--    Root world link-->
-    <link name="world"/>
+    <!-- <link name="world"/> -->
     <!-- husky base -->
     <xacro:unless value="$(arg fixed_base)">
-        <link name="husky_base_root_link"/>
+        <!-- <link name="odom"/>
         <joint name="world_joint" type="fixed">
             <parent link="world"/>
-            <child link="husky_base_root_link"/>
-        </joint>
-        <joint name="husky_base_flange" type="fixed">
+            <child link="odom"/>
+        </joint> -->
+        <!-- <joint name="husky_base_flange" type="fixed">
             <parent link="husky_base_root_link"/>
             <child link="base_link"/>
             <origin xyz="0 0 0.13228" rpy="0 0 0" />
-        </joint>
+        </joint> -->
     </xacro:unless>
     <xacro:if value="$(arg fixed_base)">
