Commit message: update a package

File: husky_panda_manipulation/data/husky_panda_mobile_model.urdf.xacro (robot description, xacro)
@@ -19,5 +19,5 @@
             <parent link="world"/>
             <child link="base_link"/>
-             <origin xyz="-0.5265965085817698 -0.2806388380571893 0.0" rpy="0.000 0.000 -0.04332860681335808"/>
+            <origin xyz="-0.5265965085817698 -0.2806388380571893 0.0" rpy="0.000 0.000 -0.04332860681335808"/>
         </joint>
     </xacro:if>

File: husky_panda_manipulation/data/husky_panda_planar.urdf (robot description, URDF)
Before this commit: robot panda, 31 links, 30 joints
Links:
- removed link panda_grasp
- link base_link: geometry collision box size=0.78992 0.5709 0.10375; collision box size=0.9874 0.5709 0.12375
- link front_bumper_link: geometry visual mesh filename=meshes/husky/bumper.dae
- link panda_hand: geometry collision box size=0.035 0.19 0.065; visual mesh filename=meshes/panda/visual/hand.dae
- link panda_leftfinger: geometry collision box size=0.0222 0.007 0.025; collision box size=0.0222 0.0145 0.018
- link panda_link0: geometry collision mesh filename=meshes/panda/collision/link0.obj; visual mesh filename=meshes/panda/visual/link0.dae
- link panda_link1: geometry collision mesh filename=meshes/panda/collision/link1.obj; visual mesh filename=meshes/panda/visual/link1.dae
- link panda_link2: geometry collision mesh filename=meshes/panda/collision/link2.obj; visual mesh filename=meshes/panda/visual/link2.dae
- link panda_link3: geometry collision mesh filename=meshes/panda/collision/link3.obj; visual mesh filename=meshes/panda/visual/link3.dae
- link panda_link4: geometry collision mesh filename=meshes/panda/collision/link4.obj; visual mesh filename=meshes/panda/visual/link4.dae
- link panda_link5: geometry collision mesh filename=meshes/panda/collision/link5.obj; visual mesh filename=meshes/panda/visual/link5.dae
- link panda_link6: geometry collision mesh filename=meshes/panda/collision/link6.obj; visual mesh filename=meshes/panda/visual/link6.dae
- link panda_link7: geometry collision mesh filename=meshes/panda/collision/link7.obj; visual mesh filename=meshes/panda/visual/link7.dae
- link panda_rightfinger: geometry collision box size=0.0222 0.007 0.025; collision box size=0.0222 0.0145 0.018
- link rear_bumper_link: geometry visual mesh filename=meshes/husky/bumper.dae
- link top_chassis_link: geometry visual mesh filename=meshes/husky/top_chassis.dae
- link top_plate_link: geometry visual mesh filename=meshes/husky/top_plate.dae
- link user_rail_link: geometry visual mesh filename=meshes/husky/user_rail.dae
Joints:
- removed joint panda_grasp_joint
- joint arm_mount_joint: origin xyz=0.25 0.0 0.0 rpy=0 0 0 -> xyz=0.25 0 0 rpy=0 0 0
- joint world_joint: origin (none) -> xyz=0 0 0 rpy=0 0 0

File: husky_panda_manipulation/data/planar_base.urdf.xacro (robot description, xacro)
@@ -6,5 +6,5 @@
             <type>transmission_interface/SimpleTransmission</type>
             <joint name="${joint_name}">
-                <hardwareInterface>hardware_interface/EffortJointInterface</hardwareInterface>
+                <hardwareInterface>hardware_interface/PositionJointInterface</hardwareInterface>
             </joint>
             <actuator name="${joint_name}_motor">
