Commit message: modify holonomic model to ridgeback

File: husky_panda_manipulation/data/husky_panda.urdf (robot description, URDF)
Before this commit: robot husky_panda, 29 links, 28 joints
Links:
- added link panda_grasp
Joints:
- added joint panda_grasp_joint: type fixed, parent panda_hand, child panda_grasp, origin xyz=0 0 0.095 rpy=0 0 0, axis 0 1 0

File: husky_panda_manipulation/data/husky_panda_mobile.urdf.xacro (robot description, xacro)
@@ -15,5 +15,5 @@
         </joint> -->
         <!-- <joint name="husky_base_flange" type="fixed">
-            <parent link="husky_base_root_link"/>
+            <parent link="base_root_link"/>
             <child link="base_link"/>
             <origin xyz="0 0 0.13228" rpy="0 0 0" />

File: husky_panda_manipulation/data/husky_panda_mobile_planar.urdf.xacro (robot description, xacro)
@@ -11,7 +11,7 @@
         <joint name="world_joint" type="fixed">
             <parent link="world"/>
-            <child link="husky_base_root_link"/>
+            <child link="base_root_link"/>
         </joint>
-        <xacro:planar_base connect_to="base_link"/>
+        <xacro:planar_base connect_to="base_link" height="0.13228"/>
     </xacro:unless>
     <xacro:if value="$(arg fixed_base)">

File: husky_panda_manipulation/data/planar_base.urdf.xacro (robot description, xacro)
@@ -13,6 +13,6 @@
         </transmission>
     </xacro:macro>
-    <xacro:macro name="planar_base" params="connect_to">
-        <link name="husky_base_root_link"/>
+    <xacro:macro name="planar_base" params="connect_to height">
+        <link name="base_root_link"/>
         <link name="x_slider">
             <inertial>
@@ -37,5 +37,5 @@
         </link>
         <joint name="x_base_joint" type="prismatic">
-            <parent link="husky_base_root_link"/>
+            <parent link="base_root_link"/>
             <child link="x_slider"/>
             <origin rpy="0 0 0" xyz="0.0 0.0 0.0"/>
@@ -66,5 +66,5 @@
             <parent link="pivot"/>
             <child link="${connect_to}"/>
-            <origin xyz="0 0 0.13228" rpy="0 0 0" />
+            <origin xyz="0 0 ${height}" rpy="0 0 0" />
         </joint>
     </xacro:macro>

File: husky_panda_manipulation/data/ridgeback_panda.urdf (robot description, URDF)
Before this commit: robot husky_panda, 30 links, 29 joints
Links:
- removed link base_footprint
- removed link base_root_link
- removed link front_bumper_link
- removed link inertial_link
- removed link pivot
- removed link rear_bumper_link
- removed link top_chassis_link
- removed link top_plate_front_link
- removed link top_plate_link
- removed link top_plate_rear_link
- removed link user_rail_link
- removed link world
- removed link x_slider
- removed link y_slider
- added link axle_link; visual mesh filename=meshes/ridgeback/axle.stl
- added link chassis_link, mass 165.304; collision mesh filename=meshes/ridgeback/body-collision.obj; visual mesh filename=meshes/ridgeback/body.stl
- added link front_cover_link; visual mesh filename=meshes/ridgeback/end-cover.stl
- added link front_left_wheel_link, mass 2.3; collision cylinder length=0.079 radius=0.0759; visual mesh filename=meshes/ridgeback/wheel.stl
- added link front_lights_link; visual mesh filename=meshes/ridgeback/lights.stl
- added link front_right_wheel_link, mass 2.3; collision cylinder length=0.079 radius=0.0759; visual mesh filename=meshes/ridgeback/wheel.stl
- added link front_rocker_link, mass 10.267; visual mesh filename=meshes/ridgeback/rocker.stl
- added link left_side_cover_link; visual mesh filename=meshes/ridgeback/side-cover.stl
- added link mid_mount
- added link panda_grasp
- added link rear_cover_link; visual mesh filename=meshes/ridgeback/end-cover.stl
- added link rear_left_wheel_link, mass 2.3; collision cylinder length=0.079 radius=0.0759; visual mesh filename=meshes/ridgeback/wheel.stl
- added link rear_lights_link; visual mesh filename=meshes/ridgeback/lights.stl
- added link rear_right_wheel_link, mass 2.3; collision cylinder length=0.079 radius=0.0759; visual mesh filename=meshes/ridgeback/wheel.stl
- added link rear_rocker_link, mass 10.267; visual mesh filename=meshes/ridgeback/rocker.stl
- added link right_side_cover_link; visual mesh filename=meshes/ridgeback/side-cover.stl
- added link top_link; collision mesh filename=meshes/ridgeback/top.obj; visual mesh filename=meshes/ridgeback/top.stl
- link base_link: geometry 
- link imu_link: mass None -> 0.001
Joints:
- removed joint base_footprint_joint
- removed joint front_bumper
- removed joint husky_base_flange
- removed joint inertial_joint
- removed joint pivot_joint
- removed joint rear_bumper
- removed joint top_chassis_joint
- removed joint top_plate_front_joint
- removed joint top_plate_joint
- removed joint top_plate_rear_joint
- removed joint user_rail
- removed joint world_joint
- removed joint x_base_joint
- removed joint y_base_joint
- added joint axle_joint: type fixed, parent chassis_link, child axle_link, origin xyz=0 0 0.05 rpy=0 0 0
- added joint base_link_joint: type fixed, parent base_link, child chassis_link, origin xyz=0 0 0 rpy=0 0 0
- added joint front_cover_link_joint: type fixed, parent chassis_link, child front_cover_link, origin xyz=0 0 0 rpy=0 0 0
- added joint front_left_wheel: type continuous, parent front_rocker_link, child front_left_wheel_link, origin xyz=0 0.2755 0 rpy=0 0 0, axis 0 1 0
- added joint front_lights_link_joint: type fixed, parent chassis_link, child front_lights_link, origin xyz=0 0 0 rpy=0 0 0
- added joint front_right_wheel: type continuous, parent front_rocker_link, child front_right_wheel_link, origin xyz=0 -0.2755 0 rpy=0 0 0, axis 0 1 0
- added joint front_rocker: type fixed, parent axle_link, child front_rocker_link, origin xyz=0.319 0 0 rpy=0 0 0, axis 1 0 0
- added joint left_side_cover_link_joint: type fixed, parent chassis_link, child left_side_cover_link, origin xyz=0 0 0 rpy=0 0 0
- added joint mid_mount_joint: type fixed, parent base_link, child mid_mount, origin xyz=0 0 0.28 rpy=0 0 0
- added joint panda_grasp_joint: type fixed, parent panda_hand, child panda_grasp, origin xyz=0 0 0.095 rpy=0 0 0, axis 0 1 0
- added joint rear_cover_link_joint: type fixed, parent chassis_link, child rear_cover_link, origin xyz=0 0 0 rpy=0 0 0
- added joint rear_left_wheel: type continuous, parent rear_rocker_link, child rear_left_wheel_link, origin xyz=0 0.2755 0 rpy=0 0 0, axis 0 1 0
- added joint rear_lights_link_joint: type fixed, parent chassis_link, child rear_lights_link, origin xyz=0 0 0 rpy=0 0 0
- added joint rear_right_wheel: type continuous, parent rear_rocker_link, child rear_right_wheel_link, origin xyz=0 -0.2755 0 rpy=0 0 0, axis 0 1 0
- added joint rear_rocker: type fixed, parent axle_link, child rear_rocker_link, origin xyz=-0.319 0 0 rpy=0 0 0, axis 1 0 0, limit effort=0 velocity=0
- added joint right_side_cover_link_joint: type fixed, parent chassis_link, child right_side_cover_link, origin xyz=0 0 0 rpy=0 0 0
- added joint top_link_joint: type fixed, parent chassis_link, child top_link, origin xyz=0 0 0 rpy=0 0 0
- joint arm_mount_joint: parent top_plate_link -> mid_mount
- joint imu_joint: origin xyz=0.19 0 0.149 rpy=0 -1.5708 3.1416 -> xyz=0.2085 -0.2902 0.1681 rpy=0 0 0; parent base_link -> chassis_link
- joint reference_link_joint: parent top_plate_link -> mid_mount

File: husky_panda_manipulation/data/ridgeback_panda_mobile_model.urdf.xacro (robot description, xacro)
@@ -4,5 +4,5 @@
     <xacro:include filename="$(find husky_panda_manipulation)/data/panda.urdf.xacro"/>
     <xacro:include filename="$(find husky_panda_manipulation)/data/planar_base.urdf.xacro"/>
-    <xacro:include filename="$(find husky_panda_manipulation)/data/husky_without_wheel.urdf.xacro"/>
+    <xacro:include filename="$(find husky_panda_manipulation)/data/ridgeback_without_wheel.urdf.xacro"/>
     <!--    Root world link-->
     <link name="world"/>
@@ -13,5 +13,5 @@
             <child link="base_root_link"/>
         </joint>
-        <xacro:planar_base connect_to="base_link" height="0.13228"/>
+        <xacro:planar_base connect_to="base_link" height="0.0259"/>
     </xacro:unless>
     <xacro:if value="$(arg fixed_base)">
@@ -24,5 +24,5 @@
     <!--Mount panda on husky-->
     <joint name="arm_mount_joint" type="fixed">
-        <parent link="top_plate_link"/>
+        <parent link="mid_mount"/>
         <child link="franka_mount_link"/>
         <origin xyz="0.25 0.0 0.0" rpy="0 0 0"/>

File: husky_panda_manipulation/data/ridgeback_panda_mobile_planar.urdf.xacro (robot description, xacro)
@@ -4,5 +4,5 @@
     <xacro:include filename="$(find husky_panda_manipulation)/data/panda.urdf.xacro"/>
     <xacro:include filename="$(find husky_panda_manipulation)/data/planar_base.urdf.xacro"/>
-    <xacro:include filename="$(find husky_panda_manipulation)/data/husky_without_wheel.urdf.xacro"/>
+    <xacro:include filename="$(find husky_panda_manipulation)/data/ridgeback.urdf.xacro"/>
     <!--    Root world link-->
     <link name="world"/>
@@ -13,5 +13,5 @@
             <child link="base_root_link"/>
         </joint>
-        <xacro:planar_base connect_to="base_link" height="0.13228"/>
+        <xacro:planar_base connect_to="base_link" height="0.0259"/>
     </xacro:unless>
     <xacro:if value="$(arg fixed_base)">
@@ -19,10 +19,10 @@
             <parent link="world"/>
             <child link="base_link"/>
-            <origin xyz="-0.5265965085817698 -0.2806388380571893 0.0" rpy="0.000 0.000 -0.04332860681335808"/>
+             <origin xyz="-0.5265965085817698 -0.2806388380571893 0.0" rpy="0.000 0.000 -0.04332860681335808"/>
         </joint>
     </xacro:if>
     <!--Mount panda on husky-->
     <joint name="arm_mount_joint" type="fixed">
-        <parent link="top_plate_link"/>
+        <parent link="mid_mount"/>
         <child link="franka_mount_link"/>
         <origin xyz="0.25 0.0 0.0" rpy="0 0 0"/>
